File: hardware/direct_sample_interface.sch (KiCad schematic (older format))
At the start: 47 parts, among them P1 VHDC_CON, P2 BNC, P3 CONN_2X2, P4 CONN_2X2, P5 CONN_4X2, P6 CONN_4X2, T1 TRANSFO4, U1 LTC2208, U2 NCP1117

Commit message: Added/finished hardware designs for direct sample PCB
Parts:
- added C25, C26, C27, C28, C29: C, ~, symbol C
- added L2: FERRITE BEAD, ~, symbol INDUCTOR
- added P7: BNC, ~, symbol BNC
- added Q1, Q2: BC856, SOT-23, symbol BC856
- added R14, R15, R16, R17, R18, R19, R20, R21: R, ~, symbol R
- added T2: TRANSFO4, ~, symbol TRANSFO4
Connections:
- net +5V: now also L2.1
- net AGND: now also U1.PPAD, C26.1, C28.2, C29.2, P7.2 (Ext), Q1.3 (C), R14.2, R16.2, R18.2, R20.2, T2.3 (PR2)
- net ENC: now also R21.2
- net ~ENC: now also R21.1
- net REF_CLK: now reaches P1.20 (CLK11)
- net REF_CLK: now also Q2.3 (C), R18.1
- new net: C27.2, Q1.1 (B), R15.2, R16.1
- new net: Q1.2 (E), Q2.2 (E), R17.2
- new net: C28.1, Q2.1 (B), R19.2, R20.1
- new net: C27.1, R14.1, T2.1 (PR1)
- new net: C25.1, P7.1 (In)
- new net: C26.2, T2.4 (S1)
- new net: C25.2, T2.5 (S2)
- new net: C29.1, L2.2, R15.1, R17.1, R19.1
Other:
- moved on the sheet: C11, C12, C13, C14, R8
